File: motor_controller.kicad_pcb (KiCad board)
At the start: 2 copper layers, 114.3 x 54.6 mm, 22 parts, among them J1 Conn_01x02, J2 Conn_01x04, J3 Conn_01x02, J4 Conn_01x04, Q1 Q_NMOS_GDS, Q10 Q_NMOS_GDS, Q11 Q_PMOS_GSD, Q12 Q_NMOS_GDS, Q2 Q_NMOS_GDS, Q3 Q_PMOS_GSD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

Commit message: Init Layout2
Parts:
- moved J2 158.8 mm to (269.1, 114.3)
- moved J1 154.8 mm to (269.1, 107.2)
- moved J3 136.7 mm to (246.0, 129.2)
- moved U2 129.4 mm to (250.3, 140.7), turned to 0 degrees
- moved U1 127.7 mm to (250.3, 129.0), turned to 0 degrees
- moved Q1 127.1 mm to (230.3, 151.0), turned to 0 degrees
- moved Q2 124.5 mm to (261.7, 126.4)
- moved R3 116.7 mm to (211.0, 151.0), turned to 0 degrees
- moved R2 98.6 mm to (201.1, 151.0), turned to 0 degrees
- moved R1 95.9 mm to (191.2, 151.0), turned to 0 degrees
- moved Q7 91.9 mm to (226.6, 125.1), turned to 0 degrees
- moved R4 90.5 mm to (221.0, 151.0)
- moved Q9 81.7 mm to (215.1, 147.2), turned to 0 degrees
- moved Q11 74.5 mm to (238.2, 125.1), turned to 0 degrees
- moved Q10 74.0 mm to (226.6, 147.2), turned to 0 degrees
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Routing:
- net CTRL_A: track 92.4 -> 0.00 mm
- net ¬CTRL_A: track 91.3 -> 0.00 mm, vias 1 -> 0
- net CTRL_B: track 87.8 -> 0.00 mm, vias 1 -> 0
- net V_ref: track 78.0 -> 0.00 mm
- net ¬CTRL_B: track 71.1 -> 0.00 mm
- net control_B: track 64.7 -> 0.00 mm
- net Net-(Q3-Pad2): track 59.6 -> 0.00 mm
- net enable_B: track 54.0 -> 0.00 mm
- net A2: track 50.4 -> 0.00 mm
- net B1: track 47.2 -> 0.00 mm
- net Net-(Q11-Pad2): track 47.0 -> 0.00 mm
- net EN_B: track 43.3 -> 0.00 mm
- net A1: track 40.3 -> 0.00 mm
- net B2: track 37.7 -> 0.00 mm
- net EN_A: track 28.1 -> 0.00 mm
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- removed copper zone on B.Cu, net GND
- removed copper zone on F.Cu, net VDC
Other:
- board outline removed
